File: Shmample/2roll.kicad_sch (KiCad schematic)
At the start: 41 parts, among them Q1 BC547, Q2 BC557, Q3 BC547, Q4 BC547, Q5 BC557, Q6 BC557, Q7 BC547, Q8 BC557, Q9 BC547, U2 358

Commit message: Big Pads
Parts:
- removed C11: 10uF, diy-nabra:cel1, symbol Device:C_Polarized
- removed R2: 100, diy-nabra:r3, symbol Device:R
- removed R23: 10k, diy-nabra:r3, symbol Device:R
- removed TP4: Hi, diy-nabra:wvout, symbol Connector:TestPoint
- R20: value 22k -> 100k
- R21: value 100k -> 10k
Connections:
- net +9V: now also RV1.3
- net Pulse: now also U2.7; no longer R22.2
- net Hi renamed RollO
- net RollO: now also R22.2; no longer U2.7

Commit message: Final revision of revision 1 before manufacture
Parts:
- removed R22: 10k, diy-nabra:r3, symbol Device:R
- R8: value 4.7k -> 470k
Connections:
- net RollO: now also C12.1, Q9.1 (C), R19.1
Changed lines of the file:
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@@
-	(wire
-		(pts
-			(xy 190.5 33.02) (xy 190.5 36.83)
-		)
-		(stroke
-			(width 0)
-			(type default)
-		)
-	)
 	(wire
 		(pts
@@
 	(wire
 		(pts
-			(xy 190.5 44.45) (xy 190.5 46.99)
+			(xy 190.5 39.37) (xy 190.5 46.99)
 		)
 		(stroke
@@
 	(global_label "RollO"
 		(shape output)
-		(at 190.5 33.02 90)
+		(at 190.5 39.37 90)
 		(fields_autoplaced yes)
 		(effects
@@
 		)
 		(property "Intersheetrefs" "${INTERSHEET_REFS}"
-			(at 190.5 24.9549 90)
+			(at 190.5 31.3049 90)
 			(effects
 				(font
@@
 	(symbol
 		(lib_id "Device:R")
-		(at 190.5 40.64 180)
-		(unit 1)
-		(exclude_from_sim no)
-		(in_bom yes)
-		(on_board yes)
-		(dnp no)
-		(property "Reference" "R22"
-			(at 193.04 39.3699 0)
-			(effects
-				(font
-					(size 1.27 1.27)
-				)
-				(justify right)
-			)
-		)
-		(property "Value" "10k"
-			(at 193.04 41.9099 0)
-			(effects
-				(font
-					(size 1.27 1.27)
-				)
-				(justify right)
-			)
-		)
-		(property "Footprint" "diy-nabra:r3"
-			(at 192.278 40.64 90)
-			(effects
-				(font
-					(size 1.27 1.27)
-				)
-				(hide yes)
-			)
-		)
-		(property "Datasheet" "~"
-			(at 190.5 40.64 0)
-			(effects
-				(font
-					(size 1.27 1.27)
-				)
-				(hide yes)
-			)
-		)
-		(property "Description" "Resistor"
-			(at 190.5 40.64 0)
-			(effects
-				(font
-					(size 1.27 1.27)
-				)
-				(hide yes)
-			)
-		)
-		(pin "2"
-		)
-		(pin "1"
-		)
-		(instances
-			(project "Shmample"
-				(path "/1cc4cbc6-6cd4-4a68-b5af-d7edf14608e3/32dd55d8-e302-418d-85c6-2e9614554d56"
-					(reference "R22")
-					(unit 1)
-				)
-			)
-		)
-	)
-	(symbol
-		(lib_id "Device:R")
 		(at 54.61 93.98 0)
 		(mirror x)
@@
 			)
 		)
-		(property "Value" "4.7k"
+		(property "Value" "470k"
 			(at 52.07 95.2499 0)
 			(effects
