File: Shmample/power.kicad_sch (KiCad schematic)
At the start: 27 parts, among them J1 Conn_01x04_Socket, U1 LM7809_TO220, U2 358, U3 4066, U4 LM324, U5 40106, U6 LM324

Commit message: Big Pads
Parts:
- U4, U6: value LM324 -> 324
Changed lines of the file:
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@@
 			)
 		)
-		(property "Value" "LM324"
+		(property "Value" "324"
 			(at 248.92 111.7599 0)
 			(effects
@@
 			)
 		)
-		(property "Value" "LM324"
+		(property "Value" "324"
 			(at 222.25 111.7599 0)
 			(effects

Commit message: Added shmatic
Parts:
- added J2: Barrel_Jack_Switch, Connector_BarrelJack:BarrelJack_Horizontal, symbol Connector:Barrel_Jack_Switch
Connections:
- net GND: now also J2.2
- net at J1.1 (Pin_1): now also J2.3; no longer D1.2 (A)
- new net: D1.2 (A), J2.1
Other:
- moved on the sheet: J1
Changed lines of the file:
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@@
 	(wire
 		(pts
+			(xy 30.48 34.29) (xy 34.29 34.29)
+		)
+		(stroke
+			(width 0)
+			(type default)
+		)
+	)
+	(wire
+		(pts
 			(xy 193.04 99.06) (xy 193.04 102.87)
 		)
@@
 	(wire
 		(pts
+			(xy 36.83 31.75) (xy 36.83 46.99)
+		)
+		(stroke
+			(width 0)
+			(type default)
+		)
+	)
+	(wire
+		(pts
 			(xy 46.99 59.69) (xy 55.88 59.69)
 		)
@@
 	(wire
 		(pts
-			(xy 46.99 46.99) (xy 46.99 49.53)
+			(xy 34.29 46.99) (xy 30.48 46.99)
 		)
 		(stroke
@@
 	(wire
 		(pts
-			(xy 194.31 30.48) (xy 198.12 30.48)
+			(xy 46.99 46.99) (xy 46.99 49.53)
 		)
 		(stroke
@@
 	(wire
 		(pts
-			(xy 118.11 46.99) (xy 118.11 49.53)
+			(xy 194.31 30.48) (xy 198.12 30.48)
 		)
 		(stroke
@@
 	(wire
 		(pts
-			(xy 34.29 46.99) (xy 36.83 46.99)
+			(xy 118.11 46.99) (xy 118.11 49.53)
 		)
 		(stroke
@@
 	(wire
 		(pts
-			(xy 34.29 54.61) (xy 43.18 54.61)
+			(xy 30.48 54.61) (xy 43.18 54.61)
 		)
 		(stroke
@@
 	(wire
 		(pts
-			(xy 34.29 52.07) (xy 43.18 52.07)
+			(xy 30.48 52.07) (xy 43.18 52.07)
+		)
+		(stroke
+			(width 0)
+			(type default)
+		)
+	)
+	(wire
+		(pts
+			(xy 34.29 34.29) (xy 34.29 46.99)
+		)
+		(stroke
+			(width 0)
+			(type default)
+		)
+	)
+	(wire
+		(pts
+			(xy 30.48 36.83) (xy 31.75 36.83)
 		)
 		(stroke
@@
 	(wire
 		(pts
-			(xy 34.29 49.53) (xy 36.83 49.53)
+			(xy 30.48 49.53) (xy 36.83 49.53)
 		)
 		(stroke
@@
 	(wire
 		(pts
+			(xy 30.48 31.75) (xy 36.83 31.75)
+		)
+		(stroke
+			(width 0)
+			(type default)
+		)
+	)
+	(wire
+		(pts
 			(xy 181.61 99.06) (xy 179.07 99.06)
 		)
@@
 	(wire
 		(pts
+			(xy 31.75 36.83) (xy 31.75 38.1)
+		)
+		(stroke
+			(width 0)
+			(type default)
+		)
+	)
+	(wire
+		(pts
 			(xy 132.08 57.15) (xy 132.08 59.69)
 		)
@@
 	(symbol
 		(lib_id "Connector:Conn_01x04_Socket")
-		(at 29.21 49.53 0)
+		(at 25.4 49.53 0)
 		(mirror y)
 		(unit 1)
@@
 		(dnp no)
 		(property "Reference" "J1"
-			(at 29.845 59.69 0)
+			(at 26.035 59.69 0)
 			(effects
 				(font
@@
 		)
 		(property "Value" "Conn_01x04_Socket"
-			(at 29.845 57.15 0)
+			(at 26.035 57.15 0)
 			(effects
 				(font
@@
 		)
 		(property "Footprint" "diy-nabra:powern"
-			(at 29.21 49.53 0)
+			(at 25.4 49.53 0)
 			(effects
 				(font
@@
 		)
 		(property "Datasheet" "~"
-			(at 29.21 49.53 0)
+			(at 25.4 49.53 0)
 			(effects
 				(font
@@
 		)
 		(property "Description" "Generic connector, single row, 01x04, script generated"
-			(at 29.21 49.53 0)
+			(at 25.4 49.53 0)
 			(effects
 				(font
@@
 	)
 	(symbol
+		(lib_id "power:GND")
+		(at 31.75 38.1 0)
+		(unit 1)
+		(exclude_from_sim no)
+		(in_bom yes)
+		(on_board yes)
+		(dnp no)
+		(fields_autoplaced yes)
+		(property "Reference" "#PWR040"
+			(at 31.75 44.45 0)
+			(effects
+				(font
+					(size 1.27 1.27)
+				)
+				(hide yes)
+			)
+		)
+		(property "Value" "GND"
+			(at 31.75 43.18 0)
+			(effects
+				(font
+					(size 1.27 1.27)
+				)
+			)
+		)
+		(property "Footprint" ""
+			(at 31.75 38.1 0)
+			(effects
+				(font
+					(size 1.27 1.27)
+				)
+				(hide yes)
+			)
+		)
+		(property "Datasheet" ""
+			(at 31.75 38.1 0)
+			(effects
+				(font
+					(size 1.27 1.27)
+				)
+				(hide yes)
+			)
+		)
+		(property "Description" "Power symbol creates a global label with name \"GND\" , ground"
+			(at 31.75 38.1 0)
+			(effects
+				(font
+					(size 1.27 1.27)
+				)
+				(hide yes)
+			)
+		)
+		(pin "1"
+		)
+		(instances
+			(project "Shmample"
+				(path "/1cc4cbc6-6cd4-4a68-b5af-d7edf14608e3/ffc6fa36-7409-4786-8dcf-d41fdc0ff090"
+					(reference "#PWR040")
+					(unit 1)
+				)
+			)
+		)
+	)
+	(symbol
 		(lib_id "4xxx:40106")
 		(at 236.22 46.99 0)
@@
 					(unit 1)
 				)
+			)
+		)
+	)
+	(symbol
+		(lib_id "Connector:Barrel_Jack_Switch")
+		(at 22.86 34.29 0)
+		(unit 1)
+		(exclude_from_sim no)
+		(in_bom yes)
+		(on_board yes)
+		(dnp no)
+		(fields_autoplaced yes)
+		(property "Reference" "J2"
+			(at 22.86 25.4 0)
+			(effects
+				(font
+					(size 1.27 1.27)
+				)
+			)
+		)
+		(property "Value" "Barrel_Jack_Switch"
+			(at 22.86 27.94 0)
+			(effects
+				(font
+					(size 1.27 1.27)
+				)
+			)
+		)
+		(property "Footprint" "Connector_BarrelJack:BarrelJack_Horizontal"
+			(at 24.13 35.306 0)
+			(effects
+				(font
+					(size 1.27 1.27)
+				)
+				(hide yes)
+			)
+		)
+		(property "Datasheet" "~"
+			(at 24.13 35.306 0)
+			(effects
+				(font
+					(size 1.27 1.27)
+				)
+				(hide yes)
+			)
+		)
+		(property "Description" "DC Barrel Jack with an internal switch"
+			(at 22.86 34.29 0)
+			(effects
+				(font
+					(size 1.27 1.27)
+				)
+				(hide yes)
+			)
+		)
+		(pin "1"
+		)
+		(pin "3"
+		)
+		(pin "2"
+		)
+		(instances
+			(project ""
+				(path "/1cc4cbc6-6cd4-4a68-b5af-d7edf14608e3/ffc6fa36-7409-4786-8dcf-d41fdc0ff090"
+					(reference "J2")
+					(unit 1)
+				)

Commit message: Final revision of revision 1 before manufacture
Parts:
- added C28: 100uF, diy-nabra:cel2, symbol Device:C_Polarized
Connections:
- net +9V: now also C28.1
- net GND: now also C28.2
- net at J1.1 (Pin_1): now also D1.2 (A), J2.1; no longer J2.3
- no-connect marks 0 -> 1
Other:
- moved on the sheet: D5, PowerPos1
