File: Shmample/power.kicad_sch (KiCad schematic)
At the start: 29 parts, among them J1 Conn_01x04_Socket, J2 Barrel_Jack_Switch, U1 LM7809_TO220, U2 358, U3 4066, U4 324, U5 40106, U6 324

Commit message: Some rejig before manufacture
Parts:
- added PowerPos2: ThePowerOut2, Connector_PinSocket_2.54mm:PinSocket_1x02_P2.54mm_Vertical, symbol Connector:Conn_01x02_Socket
Connections:
- net +9V: now also PowerPos2.1 (Pin_1)
- net GND: now also PowerPos2.2 (Pin_2)
- net at D4.1 (K), F1.1, U1.3 (VO): now also D3.2 (A); no longer D3.1 (K)
- net at C1.1, C2.1, D1.1 (K)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: now also D3.1 (K); no longer D3.2 (A)
Other:
- moved on the sheet: D3
Changed lines of the file:
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@@
 	)
 	(junction
+		(at 147.32 46.99)
+		(diameter 0)
+		(color 0 0 0 0)
+	)
+	(junction
 		(at 247.65 99.06)
 		(diameter 0)
@@
 		(color 0 0 0 0)
 	)
+	(junction
+		(at 148.59 49.53)
+		(diameter 0)
+		(color 0 0 0 0)
+	)
 	(no_connect
 		(at 30.48 34.29)
@@
 	(wire
 		(pts
+			(xy 149.86 41.91) (xy 148.59 41.91)
+		)
+		(stroke
+			(width 0)
+			(type default)
+		)
+	)
+	(wire
+		(pts
+			(xy 148.59 49.53) (xy 147.32 49.53)
+		)
+		(stroke
+			(width 0)
+			(type default)
+		)
+	)
+	(wire
+		(pts
 			(xy 36.83 31.75) (xy 36.83 46.99)
 		)
@@
 	(wire
 		(pts
+			(xy 147.32 46.99) (xy 149.86 46.99)
+		)
+		(stroke
+			(width 0)
+			(type default)
+		)
+	)
+	(wire
+		(pts
 			(xy 46.99 59.69) (xy 55.88 59.69)
 		)
@@
 	(wire
 		(pts
+			(xy 147.32 39.37) (xy 147.32 46.99)
+		)
+		(stroke
+			(width 0)
+			(type default)
+		)
+	)
+	(wire
+		(pts
 			(xy 57.15 87.63) (xy 57.15 88.9)
 		)
@@
 	(wire
 		(pts
+			(xy 149.86 39.37) (xy 147.32 39.37)
+		)
+		(stroke
+			(width 0)
+			(type default)
+		)
+	)
+	(wire
+		(pts
 			(xy 30.48 54.61) (xy 43.18 54.61)
 		)
@@
 	(wire
 		(pts
-			(xy 143.51 46.99) (xy 149.86 46.99)
+			(xy 143.51 46.99) (xy 147.32 46.99)
 		)
 		(stroke
@@
 	(wire
 		(pts
-			(xy 149.86 49.53) (xy 147.32 49.53)
+			(xy 149.86 49.53) (xy 148.59 49.53)
 		)
 		(stroke
@@
 	(wire
 		(pts
+			(xy 148.59 41.91) (xy 148.59 49.53)
+		)
+		(stroke
+			(width 0)
+			(type default)
+		)
+	)
+	(wire
+		(pts
 			(xy 30.48 31.75) (xy 36.83 31.75)
 		)
@@
 	(symbol
 		(lib_id "Diode:1N4001")
-		(at 95.25 35.56 180)
+		(at 95.25 35.56 0)
 		(unit 1)
 		(exclude_from_sim no)
@@
 					(unit 1)
 				)
+			)
+		)
+	)
+	(symbol
+		(lib_id "Connector:Conn_01x02_Socket")
+		(at 154.94 39.37 0)
+		(unit 1)
+		(exclude_from_sim no)
+		(in_bom yes)
+		(on_board yes)
+		(dnp no)
+		(fields_autoplaced yes)
+		(property "Reference" "PowerPos2"
+			(at 156.21 39.3699 0)
+			(effects
+				(font
+					(size 1.27 1.27)
+				)
+				(justify left)
+			)
+		)
+		(property "Value" "ThePowerOut2"
+			(at 156.21 41.9099 0)
+			(effects
+				(font
+					(size 1.27 1.27)
+				)
+				(justify left)
+			)
+		)
+		(property "Footprint" "Connector_PinSocket_2.54mm:PinSocket_1x02_P2.54mm_Vertical"
+			(at 154.94 39.37 0)
+			(effects
+				(font
+					(size 1.27 1.27)
+				)
+				(hide yes)
+			)
+		)
+		(property "Datasheet" "~"
+			(at 154.94 39.37 0)
+			(effects
+				(font
+					(size 1.27 1.27)
+				)
+				(hide yes)
+			)
+		)
+		(property "Description" "Generic connector, single row, 01x02, script generated"
+			(at 154.94 39.37 0)
+			(effects
+				(font
+					(size 1.27 1.27)
+				)
+				(hide yes)
+			)
+		)
+		(pin "1"
+		)
+		(pin "2"
+		)
+		(instances
+			(project "Shmample"
+				(path "/1cc4cbc6-6cd4-4a68-b5af-d7edf14608e3/ffc6fa36-7409-4786-8dcf-d41fdc0ff090"
+					(reference "PowerPos2")
+					(unit 1)
+				)
