File: Shmample/sandh.kicad_sch (KiCad schematic)
At the start: 39 parts, among them U3 4066, U4 LM324, U6 LM324, U8 4052

Commit message: Big Pads
Parts:
- U4, U6: value LM324 -> 324
Changed lines of the file:
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@@
 			)
 		)
-		(property "Value" "LM324"
+		(property "Value" "324"
 			(at 165.1 41.91 0)
 			(effects
@@
 			)
 		)
-		(property "Value" "LM324"
+		(property "Value" "324"
 			(at 77.47 129.54 0)
 			(effects
@@
 			)
 		)
-		(property "Value" "LM324"
+		(property "Value" "324"
 			(at 77.47 92.71 0)
 			(effects
@@
 			)
 		)
-		(property "Value" "LM324"
+		(property "Value" "324"
 			(at 77.47 167.64 0)
 			(effects
@@
 			)
 		)
-		(property "Value" "LM324"
+		(property "Value" "324"
 			(at 77.47 54.61 0)
 			(effects

Commit message: Added shmatic
Parts:
- TP19: value All-Out -> Select-Out
Changed lines of the file:
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@@
 			)
 		)
-		(property "Value" "All-Out"
+		(property "Value" "Select-Out"
 			(at 189.23 50.7999 90)
 			(effects

Commit message: Final revision of revision 1 before manufacture
Parts:
- added D24, D25, D26, D27: LED, diy-nabra:led, symbol Device:LED
- added R2: 1k, diy-nabra:r3, symbol Device:R
- TP12: footprint diy-nabra:wsqu2in -> diy-nabra:wsqout
Connections:
- net +9V: now also U8.3 (Y)
- net GND: now also R2.1; no longer U8.1 (Y0), U8.2 (Y2), U8.4 (Y3), U8.5 (Y1)
- new net: D24.1 (K), D25.1 (K), D26.1 (K), D27.1 (K), R2.2
- new net Y0: D24.2 (A), U8.1 (Y0)
- new net Y1: D25.2 (A), U8.5 (Y1)
- new net Y2: D27.2 (A), U8.2 (Y2)
- new net Y3: D26.2 (A), U8.4 (Y3)
- no-connect marks 1 -> 0
