File: Shmample/sandh.kicad_sch (KiCad schematic)
At the start: 44 parts, among them U3 4066, U4 324, U6 324, U8 4052

Commit message: Some rejig before manufacture
Connections:
- net GND: now also U4.3 (+)
- net at U4.1, U4.2 (-): no longer R65.1
- net at U8.13 (X): now also R65.1; no longer U4.3 (+)
Other:
- note added: "Unused Op-amp"
- moved on the sheet: R65, TP19, U4A
Changed lines of the file:
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@@
 		)
 	)
+	(text "Unused Op-amp"
+		(exclude_from_sim no)
+		(at 252.476 27.432 0)
+		(effects
+			(font
+				(size 1.27 1.27)
+			)
+		)
+	)
 	(junction
 		(at 38.1 82.55)
@@
 	)
 	(junction
-		(at 173.99 49.53)
-		(diameter 0)
-		(color 0 0 0 0)
-	)
-	(junction
 		(at 207.01 99.06)
 		(diameter 0)
@@
 	(wire
 		(pts
+			(xy 241.3 38.1) (xy 241.3 49.53)
+		)
+		(stroke
+			(width 0)
+			(type default)
+		)
+	)
+	(wire
+		(pts
 			(xy 38.1 82.55) (xy 38.1 85.09)
 		)
@@
 	(wire
 		(pts
-			(xy 38.1 146.05) (xy 38.1 147.32)
+			(xy 245.11 38.1) (xy 241.3 38.1)
 		)
 		(stroke
@@
 	(wire
 		(pts
-			(xy 58.42 82.55) (xy 58.42 85.09)
+			(xy 38.1 146.05) (xy 38.1 147.32)
 		)
 		(stroke
@@
 	(wire
 		(pts
-			(xy 58.42 82.55) (xy 69.85 82.55)
+			(xy 58.42 82.55) (xy 58.42 85.09)
 		)
 		(stroke
@@
 	(wire
 		(pts
-			(xy 22.86 157.48) (xy 24.13 157.48)
+			(xy 58.42 82.55) (xy 69.85 82.55)
 		)
 		(stroke
@@
 	(wire
 		(pts
-			(xy 68.58 162.56) (xy 68.58 172.72)
+			(xy 22.86 157.48) (xy 24.13 157.48)
 		)
 		(stroke
@@
 	(wire
 		(pts
-			(xy 153.67 46.99) (xy 157.48 46.99)
+			(xy 68.58 162.56) (xy 68.58 172.72)
 		)
 		(stroke
@@
 	(wire
 		(pts
-			(xy 156.21 57.15) (xy 173.99 57.15)
+			(xy 243.84 48.26) (xy 261.62 48.26)
 		)
 		(stroke
@@
 	(wire
 		(pts
-			(xy 173.99 49.53) (xy 175.26 49.53)
-		)
-		(stroke
-			(width 0)
-			(type default)
-		)
-	)
-	(wire
-		(pts
 			(xy 143.51 85.09) (xy 143.51 87.63)
 		)
@@
 	(wire
 		(pts
-			(xy 172.72 49.53) (xy 173.99 49.53)
+			(xy 260.35 40.64) (xy 261.62 40.64)
+		)
+		(stroke
+			(width 0)
+			(type default)
+		)
+	)
+	(wire
+		(pts
+			(xy 153.67 46.99) (xy 157.48 46.99)
 		)
 		(stroke
@@
 	(wire
 		(pts
-			(xy 157.48 52.07) (xy 156.21 52.07)
+			(xy 245.11 43.18) (xy 243.84 43.18)
 		)
 		(stroke
@@
 	(wire
 		(pts
-			(xy 173.99 57.15) (xy 173.99 49.53)
+			(xy 261.62 48.26) (xy 261.62 40.64)
 		)
 		(stroke
@@
 	(wire
 		(pts
-			(xy 156.21 52.07) (xy 156.21 57.15)
+			(xy 243.84 43.18) (xy 243.84 48.26)
 		)
 		(stroke
@@
 	(wire
 		(pts
-			(xy 182.88 49.53) (xy 184.15 49.53)
+			(xy 165.1 46.99) (xy 166.37 46.99)
 		)
 		(stroke
@@
 	(symbol
 		(lib_id "Amplifier_Operational:LM324")
-		(at 165.1 49.53 0)
+		(at 252.73 40.64 0)
 		(unit 1)
 		(exclude_from_sim no)
@@
 		(fields_autoplaced yes)
 		(property "Reference" "U4"
-			(at 165.1 39.37 0)
+			(at 252.73 30.48 0)
 			(effects
 				(font
@@
 		)
 		(property "Value" "324"
-			(at 165.1 41.91 0)
+			(at 252.73 33.02 0)
 			(effects
 				(font
@@
 		)
 		(property "Footprint" "diy-nabra:dip14"
-			(at 163.83 46.99 0)
+			(at 251.46 38.1 0)
 			(effects
 				(font
@@
 		)
 		(property "Datasheet" "http://www.ti.com/lit/ds/symlink/lm2902-n.pdf"
-			(at 166.37 44.45 0)
+			(at 254 35.56 0)
 			(effects
 				(font
@@
 		)
 		(property "Description" "Low-Power, Quad-Operational Amplifiers, DIP-14/SOIC-14/SSOP-14"
-			(at 165.1 49.53 0)
+			(at 252.73 40.64 0)
 			(effects
 				(font
@@
 	(symbol
 		(lib_id "Connector:TestPoint")
-		(at 184.15 49.53 270)
+		(at 166.37 46.99 270)
 		(unit 1)
 		(exclude_from_sim no)
@@
 		(fields_autoplaced yes)
 		(property "Reference" "TP19"
-			(at 189.23 48.2599 90)
+			(at 171.45 45.7199 90)
 			(effects
 				(font
@@
 		)
 		(property "Value" "Select-Out"
-			(at 189.23 50.7999 90)
+			(at 171.45 48.2599 90)
 			(effects
 				(font
@@
 		)
 		(property "Footprint" "diy-nabra:wsqout"
-			(at 184.15 54.61 0)
+			(at 166.37 52.07 0)
 			(effects
 				(font
@@
 		)
 		(property "Datasheet" "~"
-			(at 184.15 54.61 0)
+			(at 166.37 52.07 0)
 			(effects
 				(font
@@
 		)
 		(property "Description" "test point"
-			(at 184.15 49.53 0)
+			(at 166.37 46.99 0)
 			(effects
 				(font
@@
 	(symbol
 		(lib_id "Device:R")
-		(at 179.07 49.53 90)
+		(at 161.29 46.99 90)
 		(unit 1)
 		(exclude_from_sim no)
@@
 		(fields_autoplaced yes)
 		(property "Reference" "R65"
-			(at 179.07 43.18 90)
+			(at 161.29 40.64 90)
 			(effects
 				(font
@@
 		)
 		(property "Value" "10k"
-			(at 179.07 45.72 90)
+			(at 161.29 43.18 90)
 			(effects
 				(font
@@
 		)
 		(property "Footprint" "diy-nabra:r3"
-			(at 179.07 51.308 90)
+			(at 161.29 48.768 90)
 			(effects
 				(font
@@
 		)
 		(property "Datasheet" "~"
-			(at 179.07 49.53 0)
+			(at 161.29 46.99 0)
 			(effects
 				(font
@@
 		)
 		(property "Description" "Resistor"
-			(at 179.07 49.53 0)
+			(at 161.29 46.99 0)
 			(effects
 				(font
@@
 					(unit 1)
 				)
+			)
+		)
+	)
+	(symbol
+		(lib_id "power:GND")
+		(at 241.3 49.53 0)
+		(unit 1)
+		(exclude_from_sim no)
+		(in_bom yes)
+		(on_board yes)
+		(dnp no)
+		(fields_autoplaced yes)
+		(property "Reference" "#PWR0103"
+			(at 241.3 55.88 0)
+			(effects
+				(font
+					(size 1.27 1.27)
+				)
+				(hide yes)
+			)
+		)
+		(property "Value" "GND"
+			(at 241.3 54.61 0)
+			(effects
+				(font
+					(size 1.27 1.27)
+				)
+			)
+		)
+		(property "Footprint" ""
+			(at 241.3 49.53 0)
+			(effects
+				(font
+					(size 1.27 1.27)
+				)
+				(hide yes)
+			)
+		)
+		(property "Datasheet" ""
+			(at 241.3 49.53 0)
+			(effects
+				(font
+					(size 1.27 1.27)
+				)
+				(hide yes)
+			)
+		)
+		(property "Description" "Power symbol creates a global label with name \"GND\" , ground"
+			(at 241.3 49.53 0)
+			(effects
+				(font
+					(size 1.27 1.27)
+				)
+				(hide yes)
+			)
+		)
+		(pin "1"
+		)
+		(instances
+			(project "Shmample"
+				(path "/1cc4cbc6-6cd4-4a68-b5af-d7edf14608e3/047be123-b995-44bb-abcb-dd3aba29b22d"
+					(reference "#PWR0103")
+					(unit 1)
+				)
