File: Shmample/shift_reg.kicad_sch (KiCad schematic)
At the start: 71 parts, among them Q10 BC547, Q11 BC547, Q12 BC547, Q13 BC547, Q14 BC547, U4 LM324, U5 40106, U7 4015

Commit message: Big Pads
Parts:
- added R23: 10k, diy-nabra:r3, symbol Device:R
- added TP4: Hi, diy-nabra:wvout, symbol Connector:TestPoint
- R66: value 100k -> 22k
- U4: value LM324 -> 324
Connections:
- net MIDO2 renamed Hi
- net Hi: now also R23.1; no longer U4.10 (+)
- new net: R23.2, TP4.1
- new net MIDO: U4.10 (+)
Changed lines of the file:
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@@
 	(wire
 		(pts
+			(xy 220.98 186.69) (xy 220.98 187.96)
+		)
+		(stroke
+			(width 0)
+			(type default)
+		)
+	)
+	(wire
+		(pts
 			(xy 81.28 130.81) (xy 83.82 130.81)
 		)
@@
 	(wire
 		(pts
+			(xy 220.98 195.58) (xy 220.98 196.85)
+		)
+		(stroke
+			(width 0)
+			(type default)
+		)
+	)
+	(wire
+		(pts
 			(xy 300.99 68.58) (xy 303.53 68.58)
 		)
@@
 		)
 	)
-	(global_label "MIDO2"
+	(global_label "Hi"
 		(shape output)
 		(at 223.52 196.85 0)
@@
 		)
 		(property "Intersheetrefs" "${INTERSHEET_REFS}"
-			(at 232.3714 196.85 0)
+			(at 228.4405 196.85 0)
 			(effects
 				(font
@@
 		)
 	)
-	(global_label "MIDO2"
+	(global_label "MIDO"
 		(shape input)
 		(at 306.07 203.2 270)
@@
 		)
 		(property "Intersheetrefs" "${INTERSHEET_REFS}"
-			(at 306.07 212.0514 90)
+			(at 306.07 210.8419 90)
 			(effects
 				(font
@@
 			)
 		)
-		(property "Value" "LM324"
+		(property "Value" "324"
 			(at 212.09 189.23 0)
 			(effects
@@
 			)
 		)
-		(property "Value" "LM324"
+		(property "Value" "324"
 			(at 300.99 38.1 0)
 			(effects
@@
 			)
 		)
-		(property "Value" "100k"
+		(property "Value" "22k"
 			(at 196.85 190.4999 0)
 			(effects
@@
 	)
 	(symbol
+		(lib_id "Connector:TestPoint")
+		(at 220.98 186.69 0)
+		(unit 1)
+		(exclude_from_sim no)
+		(in_bom yes)
+		(on_board yes)
+		(dnp no)
+		(fields_autoplaced yes)
+		(property "Reference" "TP4"
+			(at 223.52 182.1179 0)
+			(effects
+				(font
+					(size 1.27 1.27)
+				)
+				(justify left)
+			)
+		)
+		(property "Value" "Hi"
+			(at 223.52 184.6579 0)
+			(effects
+				(font
+					(size 1.27 1.27)
+				)
+				(justify left)
+			)
+		)
+		(property "Footprint" "diy-nabra:wvout"
+			(at 226.06 186.69 0)
+			(effects
+				(font
+					(size 1.27 1.27)
+				)
+				(hide yes)
+			)
+		)
+		(property "Datasheet" "~"
+			(at 226.06 186.69 0)
+			(effects
+				(font
+					(size 1.27 1.27)
+				)
+				(hide yes)
+			)
+		)
+		(property "Description" "test point"
+			(at 220.98 186.69 0)
+			(effects
+				(font
+					(size 1.27 1.27)
+				)
+				(hide yes)
+			)
+		)
+		(pin "1"
+		)
+		(instances
+			(project "Shmample"
+				(path "/1cc4cbc6-6cd4-4a68-b5af-d7edf14608e3/6c85cbcb-5e2e-44d2-a46d-091f3aead2bd"
+					(reference "TP4")
+					(unit 1)
+				)
+			)
+		)
+	)
+	(symbol
 		(lib_id "Amplifier_Operational:LM324")
 		(at 314.96 198.12 0)
@@
 			)
 		)
-		(property "Value" "LM324"
+		(property "Value" "324"
 			(at 314.96 205.74 0)
 			(effects
@@
 					(unit 1)
 				)
+			)
+		)
+	)
+	(symbol
+		(lib_id "Device:R")
+		(at 220.98 191.77 180)
+		(unit 1)
+		(exclude_from_sim no)
+		(in_bom yes)
+		(on_board yes)
+		(dnp no)
+		(fields_autoplaced yes)
+		(property "Reference" "R23"
+			(at 223.52 190.4999 0)
+			(effects
+				(font
+					(size 1.27 1.27)
+				)
+				(justify right)
+			)
+		)
+		(property "Value" "10k"
+			(at 223.52 193.0399 0)
+			(effects
+				(font
+					(size 1.27 1.27)
+				)
+				(justify right)
+			)
+		)
+		(property "Footprint" "diy-nabra:r3"
+			(at 222.758 191.77 90)
+			(effects
+				(font
+					(size 1.27 1.27)
+				)
+				(hide yes)
+			)
+		)
+		(property "Datasheet" "~"
+			(at 220.98 191.77 0)
+			(effects
+				(font
+					(size 1.27 1.27)
+				)
+				(hide yes)
+			)
+		)
+		(property "Description" "Resistor"
+			(at 220.98 191.77 0)
+			(effects
+				(font
+					(size 1.27 1.27)
+				)
+				(hide yes)
+			)
+		)
+		(pin "1"
+		)
+		(pin "2"
+		)
+		(instances
+			(project "Shmample"
+				(path "/1cc4cbc6-6cd4-4a68-b5af-d7edf14608e3/6c85cbcb-5e2e-44d2-a46d-091f3aead2bd"
+					(reference "R23")
+					(unit 1)
+				)

Commit message: Final revision of revision 1 before manufacture
Parts:
- added C11, C25, C26, C27: 22uF, diy-nabra:cel1, symbol Device:C_Polarized
- added R47: 1k, diy-nabra:r3, symbol Device:R
- added R72, R73, R74: 10k, diy-nabra:r3, symbol Device:R
- R22: renamed from R47; value 1k -> 10k
- R51: value 100k -> 1M
- R59: value 22k -> 4.7k
- TP10: footprint diy-nabra:wsqout -> diy-nabra:wsqu2in
Connections:
- net GND: now also R22.2, R45.1, R46.1, R48.1, R47.1, R72.2, R73.2, R74.2; no longer D10.1 (K), D11.1 (K), D12.1 (K), D13.1 (K)
- net Q1B: now also C11.1; no longer R45.2
- net Q2B: now also C25.1; no longer R46.2
- net Q3B: now also C26.1; no longer R22.2
- net Q4A: now also C27.1; no longer R48.2
- net at D11.2 (A): now also C25.2, R72.1; no longer R46.1
- net at D12.2 (A): now also C26.2, R73.1; no longer R22.1
- net at D13.2 (A): now also C27.2, R74.1; no longer R48.1
- net at D10.2 (A): now also R22.1, C11.2; no longer R45.1
- new net: D11.1 (K), R46.2
- new net: D12.1 (K), R47.2
- new net: D13.1 (K), R48.2
- new net: D10.1 (K), R45.2
Other:
- moved on the sheet: D10, D11, D12, D13, R22, R45, R46, R48
