File: Shmample/Shmample.kicad_pcb (KiCad board)
At the start: 2 copper layers, 127 x 127 mm, 184 parts, among them J1 Conn_01x04_Socket, J2 Barrel_Jack_Switch, Q1 BC547, Q10 BC547, Q11 BC547, Q12 BC547, Q13 BC547, Q14 BC547, Q2 BC557, Q3 BC547, Q4 BC547, Q5 BC557, Q6 BC557, Q7 BC547, Q8 BC557, Q9 BC547, U1 LM7809_TO220, U2 358, U3 4066, U4 324, U5 40106, U6 324, U7 4015, U8 4052

Commit message: Some rejig before manufacture
Parts:
- added PowerPos2: ThePowerOut2, Connector_PinSocket_2.54mm:PinSocket_1x02_P2.54mm_Vertical, F.Cu at (56.1, 17.7)
- moved TP19 98.3 mm to (44.5, 27.9)
- moved R65 97.5 mm to (48.8, 32.0), turned to -152.5 degrees
- moved D3 7.62 mm to (115.6, 31.8), turned to 180 degrees
- moved U1 2.16 mm to (78.4, 23.0)
- moved R6 1.27 mm to (122.4, 122.5)
- moved R4 1.27 mm to (113.7, 122.6)
- moved C28 0.51 mm to (42.7, 22.9)
- moved PowerPos1 0.18 mm to (52.6, 17.7)
Connections:
- D3 pad 1: Net-(D3-K) -> Net-(D1-K)
- D3 pad 2: Net-(D1-K) -> Net-(D3-A)
- D4 pad 1: Net-(D3-K) -> Net-(D3-A)
- F1 pad 1: Net-(D3-K) -> Net-(D3-A)
- R65 pad 1: Net-(U4A--) -> Net-(U8-X)
- U1 pad 3: Net-(D3-K) -> Net-(D3-A)
- U4 pad 3: Net-(U4A-+) -> GND
- U8 pad 13: Net-(U4A-+) -> Net-(U8-X)
Routing:
- net Net-(U4A-+): track 119.9 -> 0.00 mm
- net Net-(D3-K): track 51.8 -> 0.00 mm
- net Net-(D3-A): track 0.00 -> 49.6 mm
- net Net-(U8-X): track 0.00 -> 8.17 mm
- net Net-(U4A--): track 8.53 -> 2.54 mm
- net +9V: track 584.8 -> 588.5 mm
- net Net-(D1-K): track 65.5 -> 63.4 mm
- net Net-(R4-Pad1): track 3.81 -> 5.08 mm
- net Net-(Q2-B): track 16.6 -> 15.4 mm
- net Net-(R65-Pad2): track 4.99 -> 5.91 mm
Other:
- board text added: "Sh'mample Design and PCB by Neil Massey Rev 1 Jun 2026"
- board text removed: "Sh'mample Design and PCB by Neil Massey Rev 1 Jan 2026"
